File: esp32.kicad_pcb (KiCad board)
At the start: 4 copper layers, 40 x 60 mm, 62 parts, among them J1 Conn_01x09_Pin, J2 ANALOG, J3 SERIAL, J4 USB_C_Receptacle_USB2.0_16P, J5 Conn_01x02_Pin, Q1 IRLML6244, Q2 IRLML6244, Q3 IRLML6244, Q4 IRLML6244, Q5 IRLML6244, Q6 BSS138, Q7 BSS138, SW1 RESET, SW2 BOOT, U1 ESP32-WROOM-32, U2 CH224K, U3 AMS1117-5.0, U4 CH340G, U5 USBLC6-2SC6, U6 AMS1117-3.3

Commit message: v1
Parts:
- renumbered C4 to C1, C6 to C11, C1 to C3, C3 to C4, C11 to C5, C9 to C6, C8 to C7, C7 to C8, C5 to C9, D2 to D1, D1 to D2, J4 to J1, J1 to J18, J5 to J2, J2 to J3, J3 to J4, JP4 to JP1, JP1 to JP4, Q7 to Q1, Q6 to Q2, Q1 to Q3, Q2 to Q5, Q3 to Q6, Q5 to Q7, R17 to R1, R14 to R10, R4 to R11, R5 to R12, R8 to R13, R6 to R14, R13 to R15, R10 to R16, R9 to R17, R7 to R18, R11 to R19, R18 to R2, R12 to R20, R1 to R21, R3 to R22, R19 to R3, R2 to R4, R15 to R7, R16 to R8, R20 to R9, TP2 to TP1, TP1 to TP2, TP5 to TP3, TP3 to TP5, U5 to U2, U4 to U3, U2 to U4, U6 to U5, U3 to U6
Connections:
- net BOOT renamed /BOOT
- net CFG1 renamed /CFG1
- net CFG2 renamed /CFG2
- net CFG3 renamed /CFG3
- net IO15 renamed /IO15
- net IO16 renamed /IO16
- net IO17 renamed /IO17
- net IO18 renamed /IO18
- net IO19 renamed /IO19
- net IO2 renamed /IO2
- net IO21 renamed /IO21
- net IO23 renamed /IO23
- net IO26 renamed /IO26
- net IO32 renamed /IO32
- net IO33 renamed /IO33
- net IO34 renamed /IO34
- net IO4 renamed /IO4
- net RESET renamed /RESET
- net SCK renamed /SCK
- net SD0 renamed /SD0
- J18 pad 9: VOUT -> VBUS
- J3 pad 6: VOUT -> VBUS
- J4 pad 2: TXD -> /TXD
- J4 pad 3: RXD -> /RXD
- R1 pad 2: VOUT -> VBUS
- R18 pad 1: TXD -> /TXD
- R20 pad 1: RXD -> /RXD
- U3 pad 16: VBUS -> +5V
- U3 pad 2: RXD -> /TXD
- U3 pad 3: TXD -> /RXD
Routing:
- net GND: track 90.0 -> 5.68 mm, vias 29 -> 38
- net VOUT: track 115.4 -> 40.5 mm, vias 1 -> 0
- net RXD: track 52.2 -> 0.00 mm, vias 2 -> 0
- net +5V: track 94.6 -> 44.1 mm, vias 5 -> 3
- net TXD: track 50.0 -> 0.00 mm, vias 2 -> 0
- net /TXD: track 0.00 -> 47.3 mm, vias 0 -> 2
- net /RXD: track 0.00 -> 45.8 mm, vias 0 -> 2
- net /IO16: track 90.0 -> 55.3 mm
- net /IO2: track 22.9 -> 0.00 mm, vias 2 -> 0
- net VBUS: track 89.6 -> 70.1 mm, vias 4 -> 0
- net /BOOT: track 44.8 -> 31.1 mm, vias 5 -> 4
- net /CFG1: track 32.7 -> 24.7 mm
- net /CFG2: track 25.6 -> 19.2 mm
- net USB_D-: track 11.3 -> 7.43 mm
- net USB_D+: track 11.0 -> 7.47 mm
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