File: esp32.kicad_sch (KiCad schematic)
At the start: 62 parts, among them J1 Conn_01x09_Pin, J2 ANALOG, J3 SERIAL, J4 USB_C_Receptacle_USB2.0_16P, J5 Conn_01x02_Pin, Q1 IRLML6244, Q2 IRLML6244, Q3 IRLML6244, Q4 IRLML6244, Q5 IRLML6244, Q6 BSS138, Q7 BSS138, SW1 RESET, SW2 BOOT, U1 ESP32-WROOM-32, U2 CH224K, U3 AMS1117-5.0, U4 CH340G, U5 USBLC6-2SC6, U6 AMS1117-3.3

Commit message: v1
Parts:
- U5: renamed from U6; footprint Package_TO_SOT_SMD:SOT-223 -> Package_TO_SOT_SMD:SOT-223-3_TabPin2
- U6: renamed from U3; footprint Package_TO_SOT_SMD:SOT-223 -> Package_TO_SOT_SMD:SOT-223-3_TabPin2
- renumbered C4 to C1, C6 to C11, C1 to C3, C3 to C4, C11 to C5, C9 to C6, C8 to C7, C7 to C8, C5 to C9, D2 to D1, D1 to D2, J4 to J1, J1 to J18, J5 to J2, J2 to J3, J3 to J4, JP4 to JP1, JP1 to JP4, Q7 to Q1, Q6 to Q2, Q1 to Q3, Q2 to Q5, Q3 to Q6, Q5 to Q7, R17 to R1, R14 to R10, R4 to R11, R5 to R12, R8 to R13, R6 to R14, R13 to R15, R10 to R16, R9 to R17, R7 to R18, R11 to R19, R18 to R2, R12 to R20, R1 to R21, R3 to R22, R19 to R3, R2 to R4, R15 to R7, R16 to R8, R20 to R9, TP2 to TP1, TP1 to TP2, TP5 to TP3, TP3 to TP5, U5 to U2, U4 to U3, U2 to U4
Connections:
- net +5V: now also U3.16 (VCC)
- net RXD: now also U3.3 (RXD); no longer U3.2 (RXD)
- net TXD: now also U3.2 (TXD); no longer U3.3 (TXD)
- net VBUS: now also J18.9 (Pin_9), J3.6 (Pin_6), R1.2; no longer U3.16 (VCC)
- net VOUT: no longer J18.9 (Pin_9), J3.6 (Pin_6), R1.2
Other:
- moved on the sheet: D2
